File: v0.1/FPGA_TB.kicad_pcb (KiCad board)
At the start: 4 copper layers, 68.6 x 53.3 mm, 111 parts, among them J1 AudioJack3, J2 AudioJack3, J3 Micro_SD_Card_Det_Hirose_DM3AT, J4 Conn_01x04, P1 USB_C_Plug_USB2.0, P2 Digital, P3 Power, P4 Digital, P5 Analog, P5 CONN_01X01, P6 CONN_01X01, P7 CONN_01X01, P8 CONN_01X01, Q1 IRLML2060, Q2 IRLML2060, Q3 IRLML2060, Q4 IRLML2060, SW1 SW_Push, U1 PCM1808PWG4, U10 W25Q32JVZP, U2 ICE40UP5K-SG48ITR, U3 FT232H, U4 93LCxxAxxOT, U5 WM8524CGEDT, U6 AP2127N-2.5, U7 APE8865N-12-HF-3, U8 AMS1117-3.3, U9 nRF52832-QFxx, X1 ASE-xxxMHz, Y1 12MHz, Y2 32MHz

Commit message: Matched some trace lenths
Parts:
- moved REF** 1.27 mm to (178.4, 101.6)
- moved Y1 0.51 mm to (143.3, 70.4), turned to 0 degrees
- moved P1 0.51 mm to (122.7, 66.3)
Routing:
- net /FLASH_IO3: track 10.3 -> 23.0 mm
- net /FLASH_IO2: track 10.3 -> 23.0 mm
- net /FLASH_CLK: track 54.0 -> 62.4 mm
- net /FET3: track 24.1 -> 31.6 mm
- net /FLASH_MOSI: track 51.2 -> 57.8 mm
- net /PINH_D7: track 19.8 -> 26.0 mm
- net Net-(C17-Pad1): track 6.65 -> 10.8 mm
- net /PINH_A4: track 28.8 -> 24.9 mm
- net /PINH_D6: track 22.2 -> 26.0 mm
- net /FET2: track 27.9 -> 31.6 mm
- net /FLASH_MISO: track 60.7 -> 64.4 mm
- net /PINH_D5: track 22.4 -> 26.0 mm
- net /FPGA_NRF1: track 23.1 -> 26.5 mm
- net /DAC_BCLK: track 36.3 -> 39.4 mm
- net Net-(C34-Pad1): track 12.9 -> 15.5 mm
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Other:
- board text removed: "1"
